File: assets/liz/liz_sensor_2_layer_v1.1/liz_sensor.kicad_pcb (KiCad board)
At the start: 2 copper layers, 25 x 40 mm, 39 parts, among them J1 USB_C_Receptacle_USB2.0_16P, U1 ESP32-S3-MINI-1-N8, U2 D3V3XA4B10LP, U5 TLV75801PDRVR

Commit message: chore: liz v1.1
Connections:
- R8 pad 1: /3V3 -> /GPIO2
- U1 pad 6: unconnected-(U1-IO2-Pad6) -> /GPIO2
Routing:
- net /GPIO2: track 0.00 -> 18.6 mm, vias 0 -> 2
- net /3V3: track 66.5 -> 64.5 mm, vias 6 -> 5
- net GND: vias 75 -> 74
Other:
- board text added: "V1.1"
- board text removed: "V1.0"
Changed lines of the file:
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@@
 	(net 40 "unconnected-(U1-RXD0-Pad40)")
 	(net 41 "unconnected-(U1-TXD0-Pad39)")
-	(net 42 "unconnected-(U1-IO2-Pad6)")
+	(net 42 "/GPIO2")
 	(net 43 "unconnected-(U1-IO37-Pad33)")
 	(net 44 "unconnected-(U1-IO39-Pad35)")
@@
 			(size 0.8 0.4)
 			(layers "F.Cu" "F.Paste" "F.Mask")
-			(net 42 "unconnected-(U1-IO2-Pad6)")
+			(net 42 "/GPIO2")
 			(pinfunction "IO2")
-			(pintype "bidirectional+no_connect")
+			(pintype "bidirectional")
 			(solder_mask_margin 0.102)
 		)
@@
 			(layers "F.Cu" "F.Paste" "F.Mask")
 			(roundrect_rratio 0.25)
-			(net 5 "/3V3")
+			(net 42 "/GPIO2")
 			(pintype "passive")
 		)
@@
 		)
 	)
-	(gr_text "V1.0"
+	(gr_text "V1.1"
 		(at 161 119.25 270)
 		(layer "B.Cu" knockout)
@@
 	)
 	(via
-		(at 150.75 94.75)
-		(size 0.6)
-		(drill 0.3)
-		(layers "F.Cu" "B.Cu")
-		(free yes)
-		(net 1)
-	)
-	(via
 		(at 146.75 92.75)
 		(size 0.6)
@@
 	)
 	(segment
-		(start 154 102.175)
-		(end 155.175 101)
-		(width 0.2)
-		(layer "F.Cu")
-		(net 5)
-	)
-	(segment
 		(start 160.75 115.5)
 		(end 160.75 114.825)
-		(width 0.24)
+		(width 0.2)
 		(layer "F.Cu")
 		(net 5)
@@
 	)
 	(segment
-		(start 154 102.5)
-		(end 154 102.175)
-		(width 0.2)
-		(layer "F.Cu")
-		(net 5)
-	)
-	(segment
 		(start 151.475 103.5)
 		(end 151.275 103.5)
@@
 		(start 160.25 116)
 		(end 160.75 115.5)
-		(width 0.24)
+		(width 0.2)
 		(layer "F.Cu")
 		(net 5)
@@
 		(net 5)
 	)
-	(via
-		(at 154 102.5)
-		(size 0.6)
-		(drill 0.3)
-		(layers "F.Cu" "B.Cu")
-		(net 5)
-	)
 	(segment
 		(start 147.488068 85.75)
@@
 		(start 154 109.75)
 		(end 160.25 116)
-		(width 0.24)
+		(width 0.2)
 		(layer "B.Cu")
 		(net 5)
@@
 	)
 	(segment
-		(start 154 102.5)
-		(end 153.75 102.25)
-		(width 0.3)
-		(layer "B.Cu")
-		(net 5)
-	)
-	(segment
 		(start 159.85 85.75)
 		(end 161.35 84.25)
@@
 	)
 	(segment
-		(start 153.75 102.25)
-		(end 151.5 102.25)
-		(width 0.3)
+		(start 154 102.5)
+		(end 153.75 102.25)
+		(width 0.2)
 		(layer "B.Cu")
 		(net 5)
@@
 		(start 154 102.5)
 		(end 154 109.75)
-		(width 0.24)
+		(width 0.2)
+		(layer "B.Cu")
+		(net 5)
+	)
+	(segment
+		(start 153.75 102.25)
+		(end 151.5 102.25)
+		(width 0.2)
 		(layer "B.Cu")
 		(net 5)
@@
 	)
 	(segment
+		(start 154.94853 101)
+		(end 155.175 101)
+		(width 0.2)
+		(layer "F.Cu")
+		(net 42)
+	)
+	(segment
+		(start 150.75 94.75)
+		(end 150.5 94.5)
+		(width 0.2)
+		(layer "F.Cu")
+		(net 42)
+	)
+	(segment
+		(start 148.5 93.75)
+		(end 148.5 89.651471)
+		(width 0.2)
+		(layer "F.Cu")
+		(net 42)
+	)
+	(segment
+		(start 149.25 94.5)
+		(end 148.5 93.75)
+		(width 0.2)
+		(layer "F.Cu")
+		(net 42)
+	)
+	(segment
+		(start 150.5 94.5)
+		(end 149.25 94.5)
+		(width 0.2)
+		(layer "F.Cu")
+		(net 42)
+	)
+	(segment
+		(start 147.048529 88.2)
+		(end 145.5 88.2)
+		(width 0.2)
+		(layer "F.Cu")
+		(net 42)
+	)
+	(segment
+		(start 148.5 89.651471)
+		(end 147.048529 88.2)
+		(width 0.2)
+		(layer "F.Cu")
+		(net 42)
+	)
+	(segment
+		(start 154.099265 100.150735)
+		(end 154.94853 101)
+		(width 0.2)
+		(layer "F.Cu")
+		(net 42)
+	)
+	(via
+		(at 154.099265 100.150735)
+		(size 0.6)
+		(drill 0.3)
+		(layers "F.Cu" "B.Cu")
+		(net 42)
+	)
+	(via
+		(at 150.75 94.75)
+		(size 0.6)
+		(drill 0.3)
+		(layers "F.Cu" "B.Cu")
+		(net 42)
+	)
+	(segment
+		(start 150.75 94.75)
+		(end 151 95)
+		(width 0.2)
+		(layer "B.Cu")
+		(net 42)
+	)
+	(segment
+		(start 151 97.05147)
+		(end 154.099265 100.150735)
+		(width 0.2)
+		(layer "B.Cu")
+		(net 42)
+	)
+	(segment
+		(start 151 95)
+		(end 151 97.05147)
+		(width 0.2)
+		(layer "B.Cu")
+		(net 42)
+	)
+	(segment
