File: assets/liz/liz_sensor_2_layer_v1.1/liz_sensor.kicad_sch (KiCad schematic)
At the start: 39 parts, among them J1 USB_C_Receptacle_USB2.0_16P, U1 ESP32-S3-MINI-1-N8, U2 D3V3XA4B10LP, U5 TLV75801PDRVR

Commit message: chore: liz v1.1
Connections:
- net 3V3: no longer R8.1
- net GPIO2: now reaches U1.6 (IO2)
- net GPIO2: now also R8.1
Other:
- moved on the sheet: C7, D1, GPIO1, R5, R8, R9
